Commit message: rework to new urdf structure

File: duatic_duadrive_interface/urdf/duadrive_interface.urdf.xacro (robot description, xacro)
@@ -22,11 +22,14 @@
 -->
 <robot xmlns:xacro="http://www.ros.org/wiki/xacro">
-<!--Base macro which represents a single duadrive-->
-<xacro:macro name="duadrive_interface_joint" params="name ethercat_address ethercat_bus mode parent_unit drive_parameter_file">
+<!--Base macro which represents a single duadrive as joint in ros2control-->
+<xacro:macro name="duadrive_interface_joint" params="name ethercat_address ethercat_bus mode parent_unit drive_parameter_file_path">
     <joint name="${name}">
       <xacro:if value="${mode != 'isaac'}">
+        <!--This is used for gazebo sim, mock hardware and real hardware-->
         <param name="ethercat_address">${ethercat_address}</param>
         <param name="ethercat_bus">${ethercat_bus}</param>
+        <!--parent unit allows us to afterwards identify which subcomponent a drive belongs to-->
         <param name="parent_unit">${parent_unit}</param>
+        <param name="drive_parameter_file_path">${drive_parameter_file_path}</param>
         <state_interface name="position">
             <!-- Slightly offset the initial position for the gazebo sim-->
