Commit message: add 'has_brake' flag into urdf

File: duatic_duadrive_interface/urdf/duadrive_interface.urdf.xacro (robot description, xacro)
@@ -23,5 +23,5 @@
 <robot xmlns:xacro="http://www.ros.org/wiki/xacro">
 <!--Base macro which represents a single duadrive as joint in ros2control-->
-<xacro:macro name="duadrive_interface_joint" params="name ethercat_address ethercat_bus mode parent_unit drive_parameter_file_path">
+<xacro:macro name="duadrive_interface_joint" params="name ethercat_address ethercat_bus mode parent_unit drive_parameter_file_path has_brake:=true">
     <joint name="${name}">
       <xacro:if value="${mode != 'isaac'}">
@@ -32,4 +32,6 @@
         <param name="parent_unit">${parent_unit}</param>
         <param name="drive_parameter_file_path">${drive_parameter_file_path}</param>
+        <!--Information if a drive is used which included a pin brake-->
+        <param name="has_brake">${has_brake}</param>
         <state_interface name="position">
             <!-- Slightly offset the initial position for the gazebo sim-->

Commit message: feat(duadrive_interface): detect brake release from motor travel
The drive only reports whether the brake solenoid is energized, not
whether the pin came out. The pin sits on the motor side of the
gearbox and limits the motor to brake_clearance of travel while it is
engaged, so the interface tracks the motor position range and reports
a new brake_released state interface once the range exceeds it.

The value latches until the stack restarts and does not depend on the
commanded solenoid state. Drives without a brake and the mock always
report released. brake_clearance is a new URDF parameter in motor rad.
Its default of 1.2 was measured on hardware to stay clear of the slot
play of an engaged pin.

File: duatic_duadrive_interface/urdf/duadrive_interface.urdf.xacro (robot description, xacro)
@@ -23,5 +23,5 @@
 <robot xmlns:xacro="http://www.ros.org/wiki/xacro">
 <!--Base macro which represents a single duadrive as joint in ros2control-->
-<xacro:macro name="duadrive_interface_joint" params="name ethercat_address ethercat_bus mode parent_unit drive_parameter_file_path has_brake:=true">
+<xacro:macro name="duadrive_interface_joint" params="name ethercat_address ethercat_bus mode parent_unit drive_parameter_file_path has_brake:=true brake_clearance:=1.2">
     <joint name="${name}">
       <xacro:if value="${mode != 'isaac'}">
@@ -34,4 +34,6 @@
         <!--Information if a drive is used which included a pin brake-->
         <param name="has_brake">${has_brake}</param>
+        <!--Motor travel in rad that an engaged brake pin still allows, used to detect a released brake-->
+        <param name="brake_clearance">${brake_clearance}</param>
         <!--Timeout in ms after which we decide that the communication with a drive has failed and we decide and error has ocurred-->
         <param name="communication_timeout">100</param>
